File: counter2/counter.brd (EAGLE design)
At the start: 127.5 x 32.8 mm, 46 parts, among them IC1 MCP1703DB, IC2 4067D, IC3 74HC154DW, J1 RJ12RIGHTANGLE-I2C, X2 8MHz, X4 MINI-USB

Commit message: set 74HC154D to gnd
Connections:
- net DMUX10: now also IC3.9; no longer IC3.10
- net DMUX9: now also IC3.10; no longer IC3.9
- net GND: now also IC3.18, IC3.19
