File: counter2/counter.brd (EAGLE design)
At the start: 127.5 x 32.8 mm, 46 parts, among them IC1 MCP1703DB, IC2 4067D, IC3 74HC154DW, J1 RJ12RIGHTANGLE-I2C, X2 8MHz, X4 MINI-USB

Commit message: add new design
Connections:
- net GND: now also IC3.18, IC3.19
Routing:
- net DMUX7: track 0.00 -> 99.0 mm, vias 0 -> 2
- net DMUX8: track 0.00 -> 83.6 mm
- net 3.3V: track 135.9 -> 208.3 mm
- net MUX7: track 0.00 -> 57.3 mm, vias 0 -> 1
- net GND: track 149.2 -> 204.5 mm, vias 0 -> 4
- net A0: track 0.00 -> 48.3 mm, vias 0 -> 1
- net DMUX5: track 24.7 -> 71.0 mm
- net MUX5: track 0.00 -> 40.6 mm, vias 0 -> 2
- net MOSI: track 0.00 -> 39.9 mm, vias 0 -> 1
- net A1: track 0.00 -> 38.1 mm, vias 0 -> 1
- net D12*: track 0.00 -> 38.0 mm, vias 0 -> 1
- net A2: track 0.00 -> 37.8 mm, vias 0 -> 1
- net MUX8: track 23.1 -> 43.7 mm
- net MUX9: track 44.5 -> 58.0 mm, vias 1 -> 2
- net DMUX11: track 38.1 -> 25.7 mm
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