File: counter2/counter.sch (EAGLE design)
At the start: 46 parts, among them IC1 MCP1703DB, IC2 4067D, IC3 74HC154DW, J1 RJ12RIGHTANGLE-I2C, X2 8MHz, X4 MINI-USB

Commit message: add new design
Connections:
- net GND: now also IC3A.G1, IC3A.G2
Changed lines of the file:
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@@
 <part name="GND10" library="supply1" library_urn="urn:adsk.eagle:library:371" deviceset="GND" device=""/>
 <part name="GND11" library="supply1" library_urn="urn:adsk.eagle:library:371" deviceset="GND" device=""/>
+<part name="GND12" library="supply1" library_urn="urn:adsk.eagle:library:371" deviceset="GND" device=""/>
 </parts>
 <sheets>
@@
 <instance part="IC3" gate="P" x="68.58" y="195.58"/>
 <instance part="P+9" gate="G$1" x="68.58" y="203.2"/>
-<instance part="GND20" gate="1" x="68.58" y="185.42"/>
+<instance part="GND20" gate="1" x="68.58" y="182.88"/>
 <instance part="GND25" gate="1" x="337.82" y="185.42"/>
 <instance part="P+21" gate="G$1" x="337.82" y="203.2"/>
@@
 <instance part="GND10" gate="1" x="215.9" y="88.9"/>
 <instance part="GND11" gate="1" x="160.02" y="88.9"/>
+<instance part="GND12" gate="1" x="78.74" y="180.34"/>
 </instances>
 <busses>
@@
 <pinref part="IC3" gate="P" pin="GND"/>
 <pinref part="GND20" gate="1" pin="GND"/>
+<wire x1="68.58" y1="185.42" x2="68.58" y2="187.96" width="0.1524" layer="91"/>
 </segment>
 <segment>
@@
 <wire x1="215.9" y1="236.22" x2="218.44" y2="236.22" width="0.1524" layer="91"/>
 </segment>
+<segment>
+<pinref part="IC3" gate="A" pin="G1"/>
+<pinref part="IC3" gate="A" pin="G2"/>
+<wire x1="78.74" y1="190.5" x2="78.74" y2="187.96" width="0.1524" layer="91"/>
+<pinref part="GND12" gate="1" pin="GND"/>
+<wire x1="78.74" y1="182.88" x2="78.74" y2="187.96" width="0.1524" layer="91"/>
+</segment>
 </net>
