File: counter3/counter.sch (EAGLE design)
At the start: 46 parts, among them IC1 MCP1703DB, IC2 4067D, IC3 74HC154DW, J1 RJ12RIGHTANGLE-I2C, X2 8MHz, X4 MINI-USB

Commit message: add new design
Parts:
- removed C1, C2: 100n, rcl:C-EUC0805
- removed CU3, CU4: 10u, rcl:C-EUC0805
- removed LDPW12: RED, adafruit:LEDCHIP-LED0805
- removed R12: 10k, rcl:R-EU_R0805
- removed RK15, RK16: 1k, rcl:R-EU_R0805
- removed RXLD: RX, adafruit:LEDCHIP-LED0805
- removed TX: TX, adafruit:LEDCHIP-LED0805
- removed U$1, U$2, U$3, U$4, U$5, U$6, U$8, U$9: GATE, custom-library:GATE
- added C11, C14, C15, C16, C17, C18, C19, C20, C21, C24, C25, C5, C6, C7, C8, C9: 10n, rcl:C-EUC0805
- added O10, O11, O12, O13, O14, O15, O16, O19, O20, O3, O4, O5, O6, O7, O8, O9: QRE1113, SparkFun:QRE1113
- added RK10, RK12, RK14, RK18, RK20, RK22, RK24, RK26, RK28, RK30, RK32, RK34, RK36, RK42, RK44, RK8: 220, resistor:R-EU_M0805
- added RK11, RK13, RK17, RK19, RK21, RK23, RK25, RK27, RK29, RK31, RK33, RK35, RK41, RK43, RK5, RK9: 1k, resistor:R-EU_M0805
- R14, R2: value 1k -> 10k
Connections:
- removed net +12V: C2.1, CU4.1, D1.A, J1.1
- removed net N$18: RK15.2, TX.A
- removed net N$2: U$1.3.3V
- removed net N$24: RK16.2, RXLD.A
- removed net N$7: LDPW12.A, R12.1
- new net 5VI2C: D1.A, J1.5
- new net RD10: O10.A, RK23.2
- new net RD11: O11.A, RK25.2
- new net RD12: O12.A, RK27.2
- new net RD13: O13.A, RK29.2
- new net RD14: O14.A, RK31.2
- new net RD15: O15.A, RK33.2
- new net RD16: O16.A, RK35.2
- new net RD19: O19.A, RK41.2
- new net RD20: O20.A, RK43.2
- new net RD3: O3.A, RK5.2
- new net RD4: O4.A, RK9.2
- new net RD5: O5.A, RK11.2
- new net RD6: O6.A, RK13.2
- new net RD7: O7.A, RK17.2
- new net RD8: O8.A, RK19.2
- new net RD9: O9.A, RK21.2
- new net Y10: C15.1, O10.C, RK24.2
- new net Y11: C16.1, O11.C, RK26.2
- new net Y12: C17.1, O12.C, RK28.2
- new net Y13: C18.1, O13.C, RK30.2
- new net Y14: C19.1, O14.C, RK32.2
- new net Y15: C20.1, O15.C, RK34.2
- new net Y16: C21.1, O16.C, RK36.2
- new net Y19: C24.1, O19.C, RK42.2
- new net Y20: C25.1, O20.C, RK44.2
- new net Y3: C5.1, O3.C, RK8.2
- new net Y4: C6.1, O4.C, RK10.2
- new net Y5: C7.1, O5.C, RK12.2
- new net Y6: C8.1, O6.C, RK14.2
- new net Y7: C9.1, O7.C, RK18.2
- new net Y8: C11.1, O8.C, RK20.2
- new net Y9: C14.1, O9.C, RK22.2
- net 3.3V: now also C11.2, C14.2, C15.2, C16.2, C17.2, C18.2, C19.2, C20.2, C21.2, C24.2, C25.2, C5.2, C6.2, C7.2, C8.2, C9.2, RK11.1, RK13.1, RK17.1, RK19.1, RK21.1, RK23.1, RK25.1, RK27.1, RK29.1, RK31.1, RK33.1, RK35.1, RK41.1, RK43.1, RK5.1, RK9.1; no longer RK15.1, RK16.1, U$3.3.3V, U$4.3.3V, U$5.3.3V, U$8.3.3V, U$9.3.3V
- net A0: now also IC3A.A; no longer IC2A.B
- net A1: now also IC3A.B; no longer IC2A.C
- net A2: now also IC3A.C; no longer IC2A.D
- net A3: now also IC3A.D
- net A4: now also IC2A.X
- net A6: now also J1.4
- net D10*: now also IC2A.INH; no longer IC3A.C
- net D11*: no longer IC3A.D
- net D12*: no longer IC2A.INH
- net D5*: now also IC2A.A
- net D6*: now also IC2A.D
- net D8*: now also IC2A.C; no longer IC3A.A
- net D9*: now also IC2A.B; no longer IC3A.B
- net DMUX1: now also IC3A.1, O3.K; no longer IC3A.7, U$1.DMUX1
- net DMUX10: now also O8.K; no longer U$5.DMUX2
- net DMUX11: now also IC3A.15, O15.K; no longer IC3A.10, U$6.DMUX1
- net DMUX12: now also IC3A.10, O16.K; no longer IC3A.11, U$6.DMUX2
- net DMUX13: now also IC3A.14, O19.K; no longer IC3A.12, U$8.DMUX1
- net DMUX14: now also IC3A.11, O20.K; no longer IC3A.13, U$8.DMUX2
- net DMUX15: now also IC3A.13, O11.K; no longer IC3A.14, U$9.DMUX1
- net DMUX16: now also IC3A.12, O12.K; no longer IC3A.15, U$9.DMUX2
- net DMUX2: now also IC3A.0, O4.K; no longer IC3A.6, U$1.DMUX2
- net DMUX3: now also IC3A.7, O5.K; no longer IC3A.5, U$2.DMUX1
- net DMUX4: now also IC3A.2, O6.K; no longer IC3A.4, U$2.DMUX2
- net DMUX5: now also IC3A.6, O9.K; no longer IC3A.3, U$3.DMUX1
- net DMUX6: now also IC3A.3, O10.K; no longer IC3A.2, U$3.DMUX2
- net DMUX7: now also IC3A.5, O13.K; no longer IC3A.1, U$4.DMUX1
- net DMUX8: now also IC3A.4, O14.K; no longer IC3A.0, U$4.DMUX2
- net DMUX9: now also O7.K; no longer U$5.DMUX1
- net GND: now also O10.E, O11.E, O12.E, O13.E, O14.E, O15.E, O16.E, O19.E, O20.E, O3.E, O4.E, O5.E, O6.E, O7.E, O8.E, O9.E; no longer C1.2, C2.2, CU3.2, CU4.2, J1.4, LDPW12.C, U$1.GND, U$2.GND, U$3.GND, U$4.GND, U$5.GND, U$6.GND, U$8.GND, U$9.GND
- net MOSI: no longer IC2A.A
- net MUX1: now also RK8.1; no longer U$1.MUX1
- net MUX10: now also RK20.1; no longer U$5.MUX2
- net MUX11: now also IC2A.X14, RK34.1; no longer IC2A.X10, U$6.MUX1
- net MUX12: now also IC2A.X15, RK36.1; no longer IC2A.X11, U$6.MUX2
- net MUX13: now also RK42.1; no longer U$8.MUX1
- net MUX14: now also RK44.1; no longer U$8.MUX2
- net MUX15: now also IC2A.X10, RK26.1; no longer IC2A.X14, U$9.MUX1
- net MUX16: now also IC2A.X11, RK28.1; no longer IC2A.X15, U$9.MUX2
- net MUX2: now also RK10.1; no longer U$1.MUX2
- net MUX3: now also IC2A.X0, RK12.1; no longer IC2A.X4, U$2.MUX1
- net MUX4: now also RK14.1; no longer U$2.MUX2
- net MUX5: now also IC2A.X1, RK22.1; no longer IC2A.X2, U$3.MUX1
- net MUX6: now also IC2A.X4, RK24.1; no longer IC2A.X3, U$3.MUX2
- net MUX7: now also IC2A.X2, RK30.1; no longer IC2A.X1, U$4.MUX1
- net MUX8: now also IC2A.X3, RK32.1; no longer IC2A.X0, U$4.MUX2
- net MUX9: now also RK18.1; no longer U$5.MUX1
- net RXLED: no longer RXLD.C
- net TXLED: no longer TX.C
- net VDD: no longer C1.1, CU3.1, R12.2
Other:
- moved on the sheet: J1
