File: counter/counter.sch (EAGLE design)
At the start: 57 parts, among them CON1 JACK_DC_BARREL, IC1 MCP1703DB, IC2 4067D, IC3 74HC154DW, J1 RJ12RIGHTANGLE-I2C, X2 8MHz, X4 MINI-USB

Commit message: counter
Parts:
- removed 12V: 12V, Headerlibrary:PINHD-1X1
- removed 3V3: (no value), Headerlibrary:PINHD-1X1
- removed C11: 100n, rcl:C-EUC0805
- removed C4: 10n, rcl:C-EUC0805
- removed CON1: JACK_DC_BARREL, lpatiny:JACK_DC_BARREL
- removed GND: GND, Headerlibrary:PINHD-1X1
- removed R10: 1K, rcl:R-EU_R0805
- removed RK1, RK2: 10K, resistor:R-EU_M0805
- removed RT2: 4.7k, resistor:R-EU_R0805
- removed SJ1: (no value), jumper:SJ
- removed U$1, U$3: QRE1113, SparkFun:QRE1113
- removed U$2: DS18B20, lpatiny:DS18B20SMALL
- added C14, C15, C18, C20, C21, C23, C25, C26, C28, C30, C32, C34, C5, C7, C8: 10n, rcl:C-EUC0805
- added I10, I12, I14, I16, I2, I4, I6, I8, O1, O11, O13, O15, O3, O5, O7, O9: QRE1113, SparkFun:QRE1113
- added RK10, RK12, RK14, RK18, RK20, RK22, RK24, RK26, RK28, RK30, RK32, RK34, RK36, RK38: 220, resistor:R-EU_M0805
- added RK11, RK13, RK17, RK19, RK21, RK23, RK25, RK27, RK29, RK31, RK33, RK35, RK37, RK9: 1k, resistor:R-EU_M0805
Connections:
- net N$12 renamed MUX2
- net N$6 renamed MUX1
- removed net N$11: IC3A.1, U$3.K
- removed net N$9: R10.2, RT2.2, U$2.DQ
- new net DMUX1: IC3A.0, O11.K
- new net DMUX10: IC3A.9, O3.K
- new net DMUX11: IC3A.10, O1.K
- new net DMUX12: I12.K, IC3A.11
- new net DMUX13: IC3A.12, O13.K
- new net DMUX14: I14.K, IC3A.13
- new net DMUX15: IC3A.14, O15.K
- new net DMUX16: I16.K, IC3A.15
- new net DMUX2: I2.K, IC3A.1
- new net DMUX3: I10.K, IC3A.2
- new net DMUX4: I4.K, IC3A.3
- new net DMUX5: IC3A.4, O9.K
- new net DMUX6: I6.K, IC3A.5
- new net DMUX7: IC3A.6, O7.K
- new net DMUX8: I8.K, IC3A.7
- new net DMUX9: IC3A.8, O5.K
- new net MUX10: IC2A.X9, RK26.1
- new net MUX11: IC2A.X10, RK28.1
- new net MUX12: IC2A.X11, RK30.1
- new net MUX13: IC2A.X12, RK32.1
- new net MUX14: IC2A.X13, RK34.1
- new net MUX15: IC2A.X14, RK36.1
- new net MUX16: IC2A.X15, RK10.1
- new net MUX3: IC2A.X2, RK38.1
- new net MUX4: IC2A.X3, RK12.1
- new net MUX5: IC2A.X4, RK14.1
- new net MUX6: IC2A.X5, RK18.1
- new net MUX7: IC2A.X6, RK20.1
- new net MUX8: IC2A.X7, RK22.1
- new net MUX9: IC2A.X8, RK24.1
- new net N$14: C7.1, O3.C, RK10.2
- new net N$17: I4.A, RK11.2
- new net N$19: C8.1, I4.C, RK12.2
- new net N$21: O9.A, RK23.2
- new net N$22: O5.A, RK13.2
- new net N$23: C14.1, O5.C, RK14.2
- new net N$27: I6.A, RK17.2
- new net N$28: C15.1, I6.C, RK18.2
- new net N$31: C21.1, O9.C, RK24.2
- new net N$32: O7.A, RK19.2
- new net N$33: C18.1, O7.C, RK20.2
- new net N$35: I10.A, RK25.2
- new net N$36: C23.1, I10.C, RK26.2
- new net N$37: I8.A, RK21.2
- new net N$38: C20.1, I8.C, RK22.2
- new net N$39: O11.A, RK27.2
- new net N$41: C25.1, O11.C, RK28.2
- new net N$43: I12.A, RK29.2
- new net N$44: C26.1, I12.C, RK30.2
- new net N$45: O13.A, RK31.2
- new net N$46: C28.1, O13.C, RK32.2
- new net N$47: I14.A, RK33.2
- new net N$48: C30.1, I14.C, RK34.2
- new net N$49: O15.A, RK35.2
- new net N$50: C32.1, O15.C, RK36.2
- new net N$51: I16.A, RK37.2
- new net N$52: C34.1, I16.C, RK38.2
- net +12V: no longer 12V.1, CON1.V+
- net 3.3V: now also C14.2, C15.2, C18.2, C20.2, C21.2, C23.2, C25.2, C26.2, C28.2, C30.2, C32.2, C34.2, C5.2, C7.2, C8.2, RK11.1, RK13.1, RK17.1, RK19.1, RK21.1, RK23.1, RK25.1, RK27.1, RK29.1, RK31.1, RK33.1, RK35.1, RK37.1, RK9.1; no longer 3V3.1, C4.2, RK1.1, RK2.1, RT2.1, U$2.VDD
- net D12*: now also IC2A.INH; no longer R10.1
- net GND: now also I10.E, I12.E, I14.E, I16.E, I2.E, I4.E, I6.E, I8.E, O1.E, O11.E, O13.E, O15.E, O3.E, O5.E, O7.E, O9.E; no longer C11.2, CON1.GND, GND.1, SJ1.1, U$1.E, U$2.GND, U$3.E
- net N$10: now also C5.1, I2.C; no longer C4.1, U$3.C
- net N$2: now also O3.A, RK9.2; no longer IC3A.0, U$1.K
- net N$4: now also O1.A; no longer U$1.A
- net N$5: now also O1.C; no longer U$1.C
- net N$8: now also I2.A; no longer U$3.A
- net RESET: no longer C11.1, SJ1.2
- net SCL: no longer RK2.2
- net SDA: no longer RK1.2
Other:
- note removed: "Power Supply"
- moved on the sheet: BKLD, C1, C2, C3, CON_ISP, CU3, CU4, CU7, CU8, CU9, D1, D2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

Commit message: Places 16 IR LED emitter/receptors on board layout with defined distances, other parts can me moved to layout board.
Connections:
- net N$10 renamed Y2
- net N$14 renamed Y3
- net N$17 renamed RD4
- net N$19 renamed Y4
- net N$2 renamed RD3
- net N$21 renamed RD9
- net N$22 renamed RD5
- net N$23 renamed Y5
- net N$27 renamed RD6
- net N$28 renamed Y6
- net N$31 renamed Y9
- net N$32 renamed RD7
- net N$33 renamed Y7
- net N$35 renamed RD10
- net N$36 renamed Y10
- net N$37 renamed RD8
- net N$38 renamed Y8
- net N$39 renamed RD11
- net N$4 renamed RD1
- net N$41 renamed Y11
- net N$43 renamed RD12
- net N$44 renamed Y12
- net N$45 renamed RD13
- net N$46 renamed Y13
- net N$47 renamed RD14
- net N$48 renamed Y14
- net N$49 renamed RD15
- net N$5 renamed Y1
- net N$50 renamed Y15
- net N$51 renamed RD16
- net N$52 renamed Y16
- net N$8 renamed RD2
- net 3.3V: now also IC2P.VDD, IC3P.VCC
- net DMUX1: now also O1.K; no longer O11.K
- net DMUX10: now also I10.K; no longer O3.K
- net DMUX11: now also O11.K; no longer O1.K
- net DMUX3: now also O3.K; no longer I10.K
- net DMUX5: now also O5.K; no longer O9.K
- net DMUX9: now also O9.K; no longer O5.K
- net GND: now also IC2P.VSS, IC3P.GND
- net MUX16: now also RK38.1; no longer RK10.1
- net MUX3: now also RK10.1; no longer RK38.1

Commit message: clean up
Parts:
- removed C1, C2: 100n, rcl:C-EUC0805
- removed C23, C26, C28, C3, C30, C32, C34: 10n, rcl:C-EUC0805
- removed CU3, CU4: 10u, rcl:C-EUC0805
- removed I10, I12, I14, I16, I2, I4, I6, I8, O1: QRE1113, SparkFun:QRE1113
- removed LDPW12: RED, adafruit:LEDCHIP-LED0805
- removed R12: 10k, rcl:R-EU_R0805
- removed RK15, RK16: 1k, rcl:R-EU_R0805
- removed RK3, RK37: 1k, resistor:R-EU_M0805
- removed RK38, RK4: 220, resistor:R-EU_M0805
- removed RXLD: RX, adafruit:LEDCHIP-LED0805
- removed TX: TX, adafruit:LEDCHIP-LED0805
- added C11, C16, C17, C19, C24, C6, C9: 10n, rcl:C-EUC0805
- added O10, O12, O14, O16, O19, O20, O4, O6, O8: QRE1113, SparkFun:QRE1113
- added RK41, RK43: 1k, resistor:R-EU_M0805
- added RK42, RK44: 220, resistor:R-EU_M0805
- R14, R2: value 1k -> 10k
Connections:
- removed net +12V: C2.1, CU4.1, D1.A, J1.1
- removed net N$18: RK15.2, TX.A
- removed net N$24: RK16.2, RXLD.A
- removed net N$7: LDPW12.A, R12.1
- removed net RD1: O1.A, RK3.2
- removed net RD2: I2.A, RK5.2
- removed net Y1: C3.1, O1.C, RK4.2
- removed net Y2: C5.1, I2.C, RK8.2
- new net 5VI2C: D1.A, J1.5
- new net RD19: O19.A, RK41.2
- new net RD20: O20.A, RK43.2
- new net Y19: C24.1, O19.C, RK42.2
- new net Y20: C25.1, O20.C, RK44.2
- net 3.3V: now also C11.2, C16.2, C17.2, C19.2, C24.2, C6.2, C9.2, RK41.1, RK43.1; no longer C23.2, C26.2, C28.2, C3.2, C30.2, C32.2, C34.2, RK15.1, RK16.1, RK3.1, RK37.1
- net A0: now also IC3A.A; no longer IC2A.B
- net A1: now also IC3A.B; no longer IC2A.C
- net A2: now also IC3A.C; no longer IC2A.D
- net A3: now also IC3A.D
- net A4: now also IC2A.X
- net A6: now also J1.4
- net D10*: now also IC2A.INH; no longer IC3A.C
- net D11*: no longer IC3A.D
- net D12*: no longer IC2A.INH
- net D5*: now also IC2A.A
- net D6*: now also IC2A.D
- net D8*: now also IC2A.C; no longer IC3A.A
- net D9*: now also IC2A.B; no longer IC3A.B
- net DMUX1: now also IC3A.1, O3.K; no longer IC3A.0, O1.K
- net DMUX10: now also O8.K; no longer I10.K
- net DMUX11: now also IC3A.15, O15.K; no longer IC3A.10, O11.K
- net DMUX12: now also IC3A.10, O16.K; no longer I12.K, IC3A.11
- net DMUX13: now also IC3A.14, O19.K; no longer IC3A.12, O13.K
- net DMUX14: now also IC3A.11, O20.K; no longer I14.K, IC3A.13
- net DMUX15: now also IC3A.13, O11.K; no longer IC3A.14, O15.K
- net DMUX16: now also IC3A.12, O12.K; no longer I16.K, IC3A.15
- net DMUX2: now also IC3A.0, O4.K; no longer I2.K, IC3A.1
- net DMUX3: now also IC3A.7, O5.K; no longer IC3A.2, O3.K
- net DMUX4: now also IC3A.2, O6.K; no longer I4.K, IC3A.3
- net DMUX5: now also IC3A.6, O9.K; no longer IC3A.4, O5.K
- net DMUX6: now also IC3A.3, O10.K; no longer I6.K, IC3A.5
- net DMUX7: now also IC3A.5, O13.K; no longer IC3A.6, O7.K
- net DMUX8: now also IC3A.4, O14.K; no longer I8.K, IC3A.7
- net DMUX9: now also O7.K; no longer O9.K
- net GND: now also IC3A.G1, IC3A.G2, O10.E, O12.E, O14.E, O16.E, O19.E, O20.E, O4.E, O6.E, O8.E; no longer C1.2, C2.2, CU3.2, CU4.2, I10.E, I12.E, I14.E, I16.E, I2.E, I4.E, I6.E, I8.E, J1.4, LDPW12.C, O1.E
- net MOSI: no longer IC2A.A
- net MUX1: now also IC2A.X6, RK8.1; no longer IC2A.X0, RK4.1
- net MUX10: now also RK20.1; no longer RK26.1
- net MUX11: now also IC2A.X14, RK34.1; no longer IC2A.X10, RK28.1
- net MUX12: now also IC2A.X15, RK36.1; no longer IC2A.X11, RK30.1
- net MUX13: now also RK42.1; no longer RK32.1
- net MUX14: now also RK44.1; no longer RK34.1
- net MUX15: now also IC2A.X10, RK26.1; no longer IC2A.X14, RK36.1
- net MUX16: now also IC2A.X11, RK28.1; no longer IC2A.X15, RK38.1
- net MUX2: now also IC2A.X7, RK10.1; no longer IC2A.X1, RK8.1
- net MUX3: now also IC2A.X0, RK12.1; no longer IC2A.X2, RK10.1
- net MUX4: now also IC2A.X5, RK14.1; no longer IC2A.X3, RK12.1
- net MUX5: now also IC2A.X1, RK22.1; no longer IC2A.X4, RK14.1
- net MUX6: now also IC2A.X4, RK24.1; no longer IC2A.X5, RK18.1
- net MUX7: now also IC2A.X2, RK30.1; no longer IC2A.X6, RK20.1
- net MUX8: now also IC2A.X3, RK32.1; no longer IC2A.X7, RK22.1
- net MUX9: now also RK18.1; no longer RK24.1
- net RD10: now also O10.A, RK23.2; no longer I10.A, RK25.2
- net RD11: now also RK25.2; no longer RK27.2
- net RD12: now also O12.A, RK27.2; no longer I12.A, RK29.2
- net RD13: now also RK29.2; no longer RK31.2
- net RD14: now also O14.A, RK31.2; no longer I14.A, RK33.2
- net RD15: now also RK33.2; no longer RK35.2
- net RD16: now also O16.A, RK35.2; no longer I16.A, RK37.2
- net RD3: now also RK5.2; no longer RK9.2
- net RD4: now also O4.A, RK9.2; no longer I4.A, RK11.2
- net RD5: now also RK11.2; no longer RK13.2
- net RD6: now also O6.A, RK13.2; no longer I6.A, RK17.2
- net RD7: now also RK17.2; no longer RK19.2
- net RD8: now also O8.A, RK19.2; no longer I8.A, RK21.2
- net RD9: now also RK21.2; no longer RK23.2
- net RXLED: no longer RXLD.C
- net TXLED: no longer TX.C
- net VDD: no longer C1.1, CU3.1, R12.2
- net Y10: now also C15.1, O10.C, RK24.2; no longer C23.1, I10.C, RK26.2
- net Y11: now also C16.1, RK26.2; no longer C25.1, RK28.2
- net Y12: now also C17.1, O12.C, RK28.2; no longer C26.1, I12.C, RK30.2
- net Y13: now also C18.1, RK30.2; no longer C28.1, RK32.2
- net Y14: now also C19.1, O14.C, RK32.2; no longer C30.1, I14.C, RK34.2
- net Y15: now also C20.1, RK34.2; no longer C32.1, RK36.2
- net Y16: now also C21.1, O16.C, RK36.2; no longer C34.1, I16.C, RK38.2
- net Y3: now also C5.1, RK8.2; no longer C7.1, RK10.2
- net Y4: now also C6.1, O4.C, RK10.2; no longer C8.1, I4.C, RK12.2
- net Y5: now also C7.1, RK12.2; no longer C14.1, RK14.2
- net Y6: now also C8.1, O6.C, RK14.2; no longer C15.1, I6.C, RK18.2
- net Y7: now also C9.1, RK18.2; no longer C18.1, RK20.2
- net Y8: now also C11.1, O8.C, RK20.2; no longer C20.1, I8.C, RK22.2
- net Y9: now also C14.1, RK22.2; no longer C21.1, RK24.2
Other:
- moved on the sheet: C18, C20, C21, C25, C5, C7, C8, J1, O11, O13, O15, O3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
