File: eagle/slaveBasic/slave-basic.brd (EAGLE design)
At the start: 99.1 x 73.7 mm, 26 parts, among them CON2 SPI, CON3 SPI, IC3 MCP1703CB, J1 RJ12RIGHTANGLE-I2C, J2 RJ12RIGHTANGLE-I2C, U3 ATMEGA328

Commit message: create slaves-i2c folder
Parts:
- removed CON2: SPI, lpatiny:TINYISP
- removed D1, D3, D4: Schottky, diode:SOD123
- removed R2: 10K, SparkFun:0603-RES
- removed RK1, RK2: 10K, resistor:M0805
- added R3: 10k, rcl:R0805
- CON3: device lpatiny:TC2030-MCP-NL -> lpatiny:TC2030-MCP
- moved C3 282.8 mm to (27.9, 27.3), turned to 180 degrees
- moved C4 274.0 mm to (28.6, 12.7)
- moved C1 257.9 mm to (19.1, 8.89)
- moved D2 243.8 mm to (19.1, 12.1)
- moved R10 240.5 mm to (45.7, 66.0), turned to 90 degrees
- moved U$1 227.7 mm to (43.8, 15.9), flipped to the bottom, turned to 90 degrees
- moved POT 219.5 mm to (90.8, 24.8), turned to 270 degrees
- moved R1 214.9 mm to (90.8, 31.1), turned to 90 degrees
- moved LCD 206.7 mm to (49.5, 55.2), flipped to the bottom
- moved IC3 55.4 mm to (19.1, 22.2), turned to 0 degrees
- moved C8 53.2 mm to (19.1, 26.0)
- moved S1 52.0 mm to (19.1, 34.3)
- moved C7 50.6 mm to (19.1, 15.2)
- moved C6 50.3 mm to (19.1, 18.4)
- moved CON3 33.7 mm to (31.1, 3.17), turned to 90 degrees
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Connections:
- removed net 3.3V: C4.1, RK1.1, RK2.1
- removed net FTDI+5V: D4.A, JP1.4
- removed net ISP+5V: CON2.VCC, CON3.5V
- removed net ISP+5V1: D2.A
- removed net N$1: C8.1, IC3.3
- removed net N$3: D1.C, D2.C, D3.C, D4.C
- new net EXT-VCC: CON3.5V, D2.A, JP1.4
- net +12V: no longer D3.A
- net +5V: now also C8.1, D2.C, IC3.3; no longer D1.A
- net GND: no longer CON2.GND
- net MISO: no longer CON2.MISO
- net MOSI: no longer CON2.MOSI
- net RESET: now also R3.1; no longer CON2.RESET, R2.1
- net SCK: no longer CON2.SCK
- net SCL: no longer RK2.2
- net SDA: no longer RK1.2
- net VCC: now also C4.1, R3.2; no longer R2.2
Routing:
- net +5V: track 0.00 -> 55.2 mm
- net RESET: track 0.00 -> 49.5 mm, vias 0 -> 2
- net VCC: track 0.00 -> 47.7 mm
- net EXT-VCC: track 0.00 -> 46.5 mm
- net SCL: track 0.00 -> 41.7 mm, vias 0 -> 1
- net GND: track 0.00 -> 36.2 mm, vias 0 -> 6
- net SDA: track 0.00 -> 33.4 mm, vias 0 -> 1
- net MISO: track 0.00 -> 33.3 mm, vias 0 -> 2
- net SCK: track 0.00 -> 28.7 mm, vias 0 -> 2
- net MOSI: track 0.00 -> 25.5 mm, vias 0 -> 2
- net +12V: track 0.00 -> 22.0 mm
- net TX: track 0.00 -> 21.5 mm, vias 0 -> 1
- net RX: track 0.00 -> 19.9 mm, vias 0 -> 1
- net DTR: track 0.00 -> 9.58 mm
- net AREF: track 0.00 -> 2.71 mm
- added copper zone on layer 16, net GND
- removed copper zone on layer 1, net GND
Other:
- board text removed: "GND"
