File: eagle/slaves-i2c/lcd-screen/slave-basic.sch (EAGLE design)
At the start: 18 parts, among them CON1 SPI, IC1 MCP1703CB, J1 RJ12RIGHTANGLE-I2C, J2 RJ12RIGHTANGLE-I2C, J3 RJ12RIGHTANGLE-I2C, U1 ATMEGA328P_TQFP

Commit message: add documentation and move lcd-screen
Parts:
- added LCD: LCD-HD447804-HOLES16X2-4-HOLES, HD44780LCD:LCD-HD447804-HOLES16X2-4-HOLES
- added POT: 10k, dp_devices:TRIMMER-3362P
- added R1: 0, rcl:R-EU_R0805
- added R2: 100, rcl:R-EU_R0805
- added U$1: EC11E, lpatiny:EC11E
Connections:
- new net N$11: LCD.A, R1.2
- new net N$2: LCD.VO, POT.2
- new net N$4: POT.1, R2.1
- net A0: now also LCD.VDD, POT.3
- net A1: now also LCD.RS
- net D10: now also R1.1
- net D2: now also U$1.A
- net D3: now also U$1.INT
- net D4: now also U$1.B
- net D5: now also LCD.E
- net D6: now also LCD.DB4
- net D7: now also LCD.DB5
- net D8: now also LCD.DB6
- net D9: now also LCD.DB7
- net GND: now also LCD.K, LCD.R/W, LCD.VSS, R2.2, U$1.CLSD, U$1.GND
Other:
- note added: "LCD 16x2"
- note added: "Rot encoder"
