File: eagle/master-simple/simple.sch (EAGLE design)
At the start: 43 parts, among them CON3 SPI, IC1 MCP1703CB, J1 RJ12RIGHTANGLE-I2C, J2 RJ12RIGHTANGLE-I2C, J3 RJ12RIGHTANGLE-I2C, X1 MINI-USB, X3 8MHz

Commit message: finalize first version of master-simple
Parts:
- removed D5: Schottky, diode:MBR0520LT
- added UART: (no value), SparkFun-Connectors:M05PTH
- L13: value RED -> BLUE
- R1: value 1k -> 10k
Connections:
- removed net +3.3: C6.1, C7.1, IC1.VO, R15.2, R31.1, U$1.VCC, U$4.AVCC, U$4.AVCC1, U$4.UVCC, U$4.VCC, U$4.VCC1
- removed net VCC-FTDI: D5.A
- new net +3V3: C6.1, C7.1, IC1.VO, R15.2, R31.1, U$1.VCC, U$4.AVCC, U$4.AVCC1, U$4.UVCC, U$4.VCC, U$4.VCC1, UART.2
- net +5V: now also UART.1
- net +XV: no longer D5.C
- net GND: now also UART.5
- net RX: now also UART.4
- net TX: now also UART.3
Other:
- note added: "I2C extensions"
- note added: "Serial extension"
- moved on the sheet: J1, J2, J3, R2, R3, R6, R7, R8, R9
