File: eagle/slaves/meteo/meteo-slave.sch (EAGLE design)
At the start: 21 parts, among them CON3 SPI, IC3 MCP1703CB, J1 RJ12RIGHTANGLE-I2C, J2 RJ12RIGHTANGLE-I2C, U3 ATMEGA328

Commit message: update meteo
Parts:
- removed J1: RJ12RIGHTANGLE-I2C, lpatiny:RJ12RIGHTANGLE-I2C
- removed U3: ATMEGA328, SparkFun:ATMEGA168
- added C2: 10u, rcl:C-EUC0805K
- added C5: 100nF, rcl:C-EUC0805K
- added D1, D3: Schottky, diode:MBR0520LT
- added J3: RJ12RIGHTANGLE-I2C, lpatiny:RJ12RIGHTANGLE-I2C
- added R12: 1M, rcl:R-EU_R0805
- added R21, R22: 4.7k, resistor:R-EU_R0805
- added R5, R7: 100, rcl:R-EU_R0805
- added R6, R9: 1K, rcl:R-EU_R0805
- added SJ1: A0, jumper:SJ
- added SJ2: A1, jumper:SJ
- added U2: (no value), RHT03_DHT-22_AM2302:RHT03_DHT-22_AM2302
- added X1: 8MHz, lpatiny:XTALNX6035
- added X2, X3: 1503_09, con-lumberg:1503_09
- C3: value 100nF -> 10u; ELECROW C49678 -> C15850; LCSC C49678 -> C15850; MPN 80-C1206C104K5R -> 77-VJ1206V106ZXQTBC
- C6: value 10u -> 100nF; ELECROW C15850 -> C49678; LCSC C15850 -> C49678; MPN 77-VJ1206V106ZXQTBC -> 80-C1206C104K5R
- C7: value 100nF -> 18pF; ELECROW C49678 -> C1797; LCSC C49678 -> C1797; MPN 80-C1206C104K5R -> 77-VJ1206A180JXXPBC
- C8: value 10u -> 18pF; ELECROW C15850 -> C1797; LCSC C15850 -> C1797; MPN 77-VJ1206V106ZXQTBC -> 77-VJ1206A180JXXPBC
- R2: value (none) -> 10k
- R4: value (none) -> 4.7k
- U$19: value MS5637 -> MS5637WIDE; device MS5637:MS5637 -> MS5637:MS5637WIDE
- U1: value (none) -> ATMEGA328P_TQFP; device RHT03_DHT-22_AM2302:RHT03_DHT-22_AM2302RA -> SparkFun-IC-Microcontroller:ATMEGA328P_TQFP
- renumbered CON3 to CON1, IC3 to IC1
Connections:
- removed net EXT-VCC: CON1.VCC, D2.A, JP1.VCC
- new net +XV: C2.1, D1.C, D2.C, D3.C, IC1.VI
- new net N$1: R22.2, R6.2, X3.2
- new net N$14: R21.1, R5.1, X2.1
- new net N$2: R22.1, R7.1, X3.1
- new net N$21: R21.2, R9.2, X2.2
- new net VCC-FTDI: D2.A, JP1.VCC
- new net VCC-ICSP: CON1.VCC, D1.A
- new net XTAL1: C8.2, R12.2, U1.PB6(XTAL1/TOSC1), X1.P$2
- new net XTAL2: C7.2, R12.1, U1.PB7(XTAL2/TOSC2), X1.P$1
- net +12V: now also J3.1; no longer J1.1
- net +5V: now also D3.A, J3.5; no longer C8.1, D2.C, IC1.VI, J1.5
- net A0: now also R1.P$2, R2.1, U1.PC0(ADC0); no longer U3.PC0(ADC0)
- net A1: now also R4.1, U$1.DQ, U1.PC1(ADC1); no longer R1.P$2, R2.1, U3.PC1(ADC1)
- net A2: now also R6.1, U1.PC2(ADC2); no longer U3.PC2(ADC2)
- net A3: now also R9.1, U1.PC3(ADC3); no longer U3.PC3(ADC3)
- net A6: now also SJ1.1, U1.ADC6; no longer U3.ADC6
- net A7: now also SJ2.1, U1.ADC7; no longer U3.ADC7
- net AREF: now also C1.1, U1.AREF; no longer C3.1, U3.AREF
- net D10: now also R4.2, R5.2, R7.2, U$1.VCC, U1.PB2(SS/OC1B); no longer U3.PB2(SS/OC1B)
- net D2: now also U1.PD2(INT0); no longer U3.PD2(INT0)
- net D3: now also U1.PD3(INT1); no longer U3.PD3(INT1)
- net D4: now also U1.PD4(XCK/T0); no longer U3.PD4(XCK/T0)
- net D5: now also R1.P$1, U1.PD5(T1); no longer U1.DATA, U3.PD5(T1)
- net D6: now also U1.PD6(AIN0), U2.DATA; no longer R4.1, U$1.DQ, U3.PD6(AIN0)
- net D7: now also U1.PD7(AIN1), U2.VDD; no longer U3.PD7(AIN1)
- net D8: now also U$19.SCL, U1.PB0(ICP); no longer U3.PB0(ICP)
- net D9: now also U$19.SDA, U1.PB1(OC1A); no longer U3.PB1(OC1A)
- net DTR: now also C6.1; no longer C1.1
- net GND: now also C1.2, C2.2, C5.2, C7.1, C8.1, J3.4, J3.6, SJ1.2, SJ2.2, U1.AGND, U2.GND, X2.3, X3.3; no longer C6.2, C7.2, C8.2, J1.4, J1.6, U3.AGND, U3.GND@1, U3.GND@2
- net MISO: now also U1.PB4(MISO); no longer U3.PB4(MISO)
- net MOSI: now also U1.PB3(MOSI/OC2); no longer U3.PB3(MOSI/OC2)
- net RESET: now also C6.2, U1.PC6(/RESET); no longer C1.2, U3.PC6(/RESET)
- net RX: now also U1.PD0(RXD); no longer U3.PD0(RXD)
- net SCK: now also U1.PB5(SCK); no longer U3.PB5(SCK)
- net SCL: now also J3.2, U1.PC5(ADC5/SCL); no longer J1.2, U$19.SCL, U3.PC5(ADC5/SCL)
- net SDA: now also J3.3, U1.PC4(ADC4/SDA); no longer J1.3, U$19.SDA, U3.PC4(ADC4/SDA)
- net TX: now also U1.PD1(TXD); no longer U3.PD1(TXD)
- net VCC: now also C3.1, C5.1, U1.AVCC, U1.VCC; no longer C6.1, C7.1, R1.P$1, R4.2, U$1.VCC, U1.VDD, U3.AVCC, U3.VCC@1, U3.VCC@2
Other:
- note added: "One wire"
- moved on the sheet: C1, C3, C4, C6, C7, C8, D2, J2, R1, R2, R3, R4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
