File: meteo-i2c/eagle/meteo/meteo-slave.sch (EAGLE design)
At the start: 37 parts, among them CON1 SPI, IC1 MCP1703CB, J2 RJ12RIGHTANGLE-I2C, J3 RJ12RIGHTANGLE-I2C, U1 ATMEGA328P_TQFP, X1 8MHz, X2 1503_09, X3 1503_09

Commit message: revert to resistor for LDR to be able to tune
Parts:
- added R2: 10k, resistor:R-EU_R0805
- R19: value 100k -> 1M
Connections:
- net A0: now also R2.1
- net D5: now also R1.P$1
- net GND: now also R2.2; no longer R1.P$1
Other:
- moved on the sheet: R1
Changed lines of the file:
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@@
 </part>
 <part name="R1" library="SparkFun" deviceset="PHOTOCELL" device="PTH"/>
+<part name="R2" library="resistor" library_urn="urn:adsk.eagle:library:348" deviceset="R-EU_" device="R0805" value="10k"/>
+<part name="GND2" library="supply1" library_urn="urn:adsk.eagle:library:371" deviceset="GND" device=""/>
 <part name="U$1" library="Ava" deviceset="DS1820" device="TO92"/>
 <part name="R4" library="resistor" library_urn="urn:adsk.eagle:library:348" deviceset="R-EU_" device="R0805" value="4.7k"/>
@@
 <attribute name="LCSC" value="C17514"/>
 </part>
-<part name="R19" library="rcl" deviceset="R-EU_" device="R0805" value="100k">
+<part name="R19" library="rcl" deviceset="R-EU_" device="R0805" value="1M">
 <attribute name="ELECROW" value="C17514"/>
 <attribute name="LCSC" value="C17514"/>
@@
 </part>
 <part name="GND7" library="supply1" library_urn="urn:adsk.eagle:library:371" deviceset="GND" device=""/>
-<part name="GND9" library="supply1" library_urn="urn:adsk.eagle:library:371" deviceset="GND" device=""/>
 </parts>
 <sheets>
@@
 <attribute name="LCSC" x="124.46" y="99.06" size="1.778" layer="96" rot="MR90" display="off"/>
 </instance>
-<instance part="R1" gate="G$1" x="193.04" y="22.86" rot="R90"/>
+<instance part="R1" gate="G$1" x="193.04" y="15.24" rot="R90"/>
+<instance part="R2" gate="G$1" x="193.04" y="38.1" rot="R90"/>
+<instance part="GND2" gate="1" x="195.58" y="45.72" rot="R90"/>
 <instance part="U$1" gate="G$1" x="160.02" y="35.56"/>
 <instance part="R4" gate="G$1" x="170.18" y="25.4" rot="R90"/>
@@
 <attribute name="VALUE" x="254.635" y="140.335" size="1.27" layer="96"/>
 </instance>
-<instance part="GND9" gate="1" x="193.04" y="10.16"/>
 </instances>
 <busses>
@@
 </segment>
 <segment>
+<pinref part="R2" gate="G$1" pin="2"/>
+<pinref part="GND2" gate="1" pin="GND"/>
+<wire x1="193.04" y1="45.72" x2="193.04" y2="43.18" width="0.1524" layer="91"/>
+</segment>
+<segment>
 <pinref part="U$1" gate="G$1" pin="GND"/>
 <pinref part="GND4" gate="1" pin="GND"/>
@@
 <junction x="256.54" y="144.78"/>
 <pinref part="GND7" gate="1" pin="GND"/>
-</segment>
-<segment>
-<pinref part="R1" gate="G$1" pin="P$1"/>
-<wire x1="193.04" y1="12.7" x2="193.04" y2="15.24" width="0.1524" layer="91"/>
-<label x="193.04" y="12.7" size="1.778" layer="95"/>
-<pinref part="GND9" gate="1" pin="GND"/>
 </segment>
 </net>
@@
 <segment>
 <pinref part="R1" gate="G$1" pin="P$2"/>
-<wire x1="193.04" y1="30.48" x2="193.04" y2="35.56" width="0.1524" layer="91"/>
-<wire x1="187.96" y1="35.56" x2="193.04" y2="35.56" width="0.1524" layer="91"/>
-<label x="185.42" y="35.56" size="1.778" layer="95" rot="R90"/>
+<pinref part="R2" gate="G$1" pin="1"/>
+<wire x1="193.04" y1="22.86" x2="193.04" y2="27.94" width="0.1524" layer="91"/>
+<wire x1="193.04" y1="27.94" x2="193.04" y2="33.02" width="0.1524" layer="91"/>
+<wire x1="187.96" y1="27.94" x2="193.04" y2="27.94" width="0.1524" layer="91"/>
+<junction x="193.04" y="27.94"/>
+<label x="185.42" y="27.94" size="1.778" layer="95" rot="R90"/>
 </segment>
 </net>
@@
 <pinref part="U1" gate="U1" pin="PD5(T1)"/>
 </segment>
-</net>
+<segment>
+<pinref part="R1" gate="G$1" pin="P$1"/>
+<wire x1="193.04" y1="5.08" x2="193.04" y2="7.62" width="0.1524" layer="91"/>
+<label x="193.04" y="5.08" size="1.778" layer="95"/>
+</segment>
+</net>
