File: master-simple/eagle/simple.brd (EAGLE design)
At the start: 75 x 43.3 mm, 43 parts, among them CON3 SPI, IC1 MCP1703CB, J1 RJ12RIGHTANGLE-I2C, J2 RJ12RIGHTANGLE-I2C, J3 RJ12RIGHTANGLE-I2C, X1 MINI-USB, X3 8MHz

Commit message: Update README.md
Parts:
- added R10, R12: 4.7k, resistor:R0805
Connections:
- net +3V3: now also R10.1, R12.1
- net SCL: now also R10.2
- net SDA: now also R12.2
Changed lines of the file:
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@@
 </element>
 <element name="UART" library="SparkFun-Connectors" package="1X05" value="" x="4.445" y="24.765" rot="R270"/>
+<element name="R10" library="resistor" library_urn="urn:adsk.eagle:library:348" package="R0805" package3d_urn="urn:adsk.eagle:package:26059/1" value="4.7k" x="-2.54" y="-3.81"/>
+<element name="R12" library="resistor" library_urn="urn:adsk.eagle:library:348" package="R0805" package3d_urn="urn:adsk.eagle:package:26059/1" value="4.7k" x="-2.54" y="-10.16"/>
 </elements>
 <signals>
@@
 <wire x1="19.77" y1="14.3" x2="20.65" y2="14.3" width="0.4064" layer="1"/>
 <wire x1="20.65" y1="14.3" x2="21.59" y2="15.24" width="0.4064" layer="1"/>
+<contactref element="R12" pad="2"/>
+<wire x1="-1.59" y1="-10.16" x2="19.77" y2="14.3" width="0" layer="19" extent="1-1"/>
 </signal>
 <signal name="SCL">
@@
 <wire x1="21.755" y1="13.5" x2="22.86" y2="14.605" width="0.4064" layer="1"/>
 <wire x1="22.86" y1="14.605" x2="22.86" y2="20.32" width="0.4064" layer="1"/>
+<contactref element="R10" pad="2"/>
+<wire x1="-1.59" y1="-3.81" x2="11.43" y2="20.32" width="0" layer="19" extent="1-1"/>
 </signal>
 <signal name="TX">
@@
 <wire x1="4.445" y1="22.225" x2="8.17" y2="18.5" width="0.4064" layer="1"/>
 <wire x1="8.17" y1="18.5" x2="8.17" y2="16.7" width="0.4064" layer="1"/>
+<contactref element="R10" pad="1"/>
+<contactref element="R12" pad="1"/>
+<wire x1="-3.49" y1="-3.81" x2="-3.49" y2="-10.16" width="0" layer="19" extent="1-1"/>
+<wire x1="1.905" y1="8.89" x2="-3.49" y2="-3.81" width="0" layer="19" extent="1-1"/>
 </signal>
 </signals>
