File: weather-i2c/eagle/meteo/meteo-slave.brd (EAGLE design)
At the start: 49.5 x 49.5 mm, 39 parts, among them CON1 SPI, IC1 MCP1703CB, J2 RJ12RIGHTANGLE-I2C, J3 RJ12RIGHTANGLE-I2C, U1 ATMEGA328P_TQFP, X1 8MHz, X2 1503_09, X3 1503_09

Commit message: weather-i2c: cleanup v1.1
Parts:
- added R10, R11: 4.7k, resistor:R0805
- moved R8 69.9 mm to (42.5, 29.2), turned to 270 degrees
- moved C11 63.3 mm to (40.0, 29.2), turned to 270 degrees
- moved R19 57.2 mm to (37.5, 29.2), turned to 270 degrees
- moved R18 50.8 mm to (34.9, 29.2), turned to 90 degrees
- moved R6 0.64 mm to (28.6, 40.0)
- moved R9 0.64 mm to (12.7, 40.0)
- moved X2 0.64 mm to (20.3, 48.9)
- moved X3 0.64 mm to (36.2, 48.9)
- moved J2 0.64 mm to (3.81, 29.8)
- moved J3 0.64 mm to (3.81, 14.0)
- moved R21 0.63 mm to (12.7, 43.8)
- moved R22 0.63 mm to (28.6, 43.8)
- moved R5 0.63 mm to (12.7, 47.6)
- moved R7 0.63 mm to (28.6, 47.6), turned to 180 degrees
Connections:
- net D8: now also R10.1
- net D9: now also R11.1
- net VCC: now also R10.2, R11.2
Routing:
- net +5V: track 56.9 -> 87.3 mm, vias 0 -> 1
- net D6: track 15.1 -> 26.1 mm
- net A6: track 4.52 -> 13.6 mm, vias 1 -> 2
- net D8: track 6.06 -> 11.7 mm
- net D7: track 16.4 -> 21.9 mm
- net GND: track 32.5 -> 35.8 mm, vias 12 -> 13
- net D9: track 6.76 -> 9.98 mm
- net D10: track 70.6 -> 73.2 mm, vias 0 -> 3
- net VCC: track 63.9 -> 65.4 mm, vias 2 -> 0
- net A0: track 54.2 -> 52.9 mm, vias 4 -> 2
- net A3: track 24.3 -> 25.0 mm
- net A2: track 17.6 -> 18.3 mm
- net SDA: track 33.8 -> 34.4 mm
Other:
- board text added: "Slave I2C - Meteo V1.1.0"
