File: scale-i2c/eagle/scale-slave.brd (EAGLE design)
At the start: 49.5 x 49.5 mm, 41 parts, among them CON1 SPI, IC1 MCP1703CB, J2 RJ12RIGHTANGLE-I2C, J3 RJ12RIGHTANGLE-I2C, U1 ATMEGA328P_TQFP, U2 HX711, X1 8MHz

Commit message: Labels positioned scale board
Parts:
- D1, D2, D3: value Schottky -> Schottky||
