File: scale-i2c/eagle/scale-slave.brd (EAGLE design)
At the start: 49.5 x 49.5 mm, 41 parts, among them CON1 SPI, IC1 MCP1703CB, J2 RJ12RIGHTANGLE-I2C, J3 RJ12RIGHTANGLE-I2C, U1 ATMEGA328P_TQFP, U2 HX711, X1 8MHz

Commit message: correct resistor for voltage check
Parts:
- R19: value 1M -> 220k
Changed lines of the file:
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@@
 <attribute name="VALUE" x="20.955" y="36.195" size="1.27" layer="27" rot="R180"/>
 </element>
-<element name="R19" library="rcl" package="R0805" value="1M" x="16.51" y="38.1" smashed="yes">
+<element name="R19" library="rcl" package="R0805" value="220k" x="16.51" y="38.1" smashed="yes">
 <attribute name="ELECROW" value="C17514" x="16.51" y="38.1" size="1.778" layer="27" display="off"/>
 <attribute name="LCSC" value="C17514" x="16.51" y="38.1" size="1.778" layer="27" display="off"/>
