File: scale-i2c/eagle/hx711-RJ12-board.brd (EAGLE design)
At the start: 44.5 x 27.9 mm, 17 parts, among them J8 RJ123.3, U1 HX711

Commit message: final scale version
Parts:
- moved 20K 52.4 mm to (36.5, 24.4)
- moved 8.2K 52.4 mm to (32.7, 24.4)
- moved C13 52.4 mm to (37.5, 21.6)
- moved C14 52.4 mm to (28.6, 24.1)
- moved C15 52.4 mm to (24.8, 19.1)
- moved CU1 52.4 mm to (34.9, 14.6)
- moved J8 52.4 mm to (11.4, 14.0)
- moved RK5 52.4 mm to (37.8, 13.7)
- moved RL1 52.4 mm to (25.1, 22.0)
- moved RL2 52.4 mm to (21.9, 13.7)
- moved SJ2 52.4 mm to (36.8, 17.8)
- moved SJ3 52.4 mm to (36.1, 7.89)
- moved U1 52.4 mm to (28.6, 14.0)
- moved BJ1 52.4 mm to (33.0, 19.7)
- moved C12 52.4 mm to (40.0, 10.8)
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Other:
- board text removed: "+"
- board text removed: "1"
- board text removed: "BLK"
- board text removed: "BeeMoS Master V 1.0"
- board text removed: "BeeMoS Master V1.0"
- board text removed: "GND"
