File: scale-i2c/eagle/scale-slave.sch (EAGLE design)
At the start: 39 parts, among them CON1 SPI, IC1 MCP1703CB, J2 RJ12RIGHTANGLE-I2C, J3 RJ12RIGHTANGLE-I2C, U1 ATMEGA328P_TQFP, U2 HX711, X1 8MHz

Commit message: final scale
Parts:
- removed SJ1: A0, jumper:SJ
- added C13: 100nF, rcl:C-EUC0805K
- added R18, R19: 1M, rcl:R-EU_R0805
Connections:
- net +5V: now also R18.2
- net A6: now also C13.2, R18.1, R19.2; no longer SJ1.1
- net GND: now also C13.1, R19.1; no longer SJ1.2
Other:
- moved on the sheet: 20K, 8.2K, BJ1, C1, C10, C11, C12, C2, C3, C4, C5, C6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

Commit message: final scale version
Parts:
- D1, D2, D3: value Schottky -> Schottky||
Changed lines of the file:
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@@
 <?xml version="1.0" encoding="utf-8"?>
 <!DOCTYPE eagle SYSTEM "eagle.dtd">
-<eagle version="9.0.1">
+<eagle version="8.7.1">
 <drawing>
 <settings>
@@
 <part name="P+10" library="supply1" library_urn="urn:adsk.eagle:library:371" deviceset="+12V" device=""/>
 <part name="P+5" library="supply1" library_urn="urn:adsk.eagle:library:371" deviceset="+12V" device=""/>
-<part name="D1" library="diode" library_urn="urn:adsk.eagle:library:210" deviceset="MBR0520LT" device="" package3d_urn="urn:adsk.eagle:package:43420/1" value="Schottky">
+<part name="D1" library="diode" library_urn="urn:adsk.eagle:library:210" deviceset="MBR0520LT" device="" package3d_urn="urn:adsk.eagle:package:43420/1" value="Schottky||">
 <attribute name="LCSC" value="C82544"/>
 <attribute name="MPN" value="621-1N5819HW-F"/>
@@
 </part>
 <part name="U1" library="SparkFun-IC-Microcontroller" deviceset="ATMEGA328P_TQFP" device="" value="ATMEGA328P_TQFP"/>
-<part name="D2" library="diode" library_urn="urn:adsk.eagle:library:210" deviceset="MBR0520LT" device="" package3d_urn="urn:adsk.eagle:package:43420/1" value="Schottky">
+<part name="D2" library="diode" library_urn="urn:adsk.eagle:library:210" deviceset="MBR0520LT" device="" package3d_urn="urn:adsk.eagle:package:43420/1" value="Schottky||">
 <attribute name="LCSC" value="C82544"/>
 <attribute name="MPN" value="621-1N5819HW-F"/>
 </part>
-<part name="D3" library="diode" library_urn="urn:adsk.eagle:library:210" deviceset="MBR0520LT" device="" package3d_urn="urn:adsk.eagle:package:43420/1" value="Schottky">
+<part name="D3" library="diode" library_urn="urn:adsk.eagle:library:210" deviceset="MBR0520LT" device="" package3d_urn="urn:adsk.eagle:package:43420/1" value="Schottky||">
 <attribute name="LCSC" value="C82544"/>
 <attribute name="MPN" value="621-1N5819HW-F"/>
