File: weather-i2c/eagle/meteo-slave.brd (EAGLE design)
At the start: 49.5 x 49.5 mm, 41 parts, among them CON1 SPI, IC1 MCP1703CB, J2 RJ12RIGHTANGLE-I2C, J3 RJ12RIGHTANGLE-I2C, U1 ATMEGA328P_TQFP, X1 8MHz, X2 1503_09, X3 1503_09

Commit message: weather-i2c: fix voltage check resistor value
Parts:
- R19: value 1M -> 220k
Changed lines of the file:
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@@
 <?xml version="1.0" encoding="utf-8"?>
 <!DOCTYPE eagle SYSTEM "eagle.dtd">
-<eagle version="9.0.0">
+<eagle version="9.1.0">
 <drawing>
 <settings>
@@
 <param name="checkStop" value="0"/>
 <param name="checkValues" value="0"/>
+<param name="checkNames" value="1"/>
+<param name="checkWireStubs" value="1"/>
+<param name="checkPolygonWidth" value="0"/>
 <param name="useDiameter" value="13"/>
 <param name="maxErrors" value="50"/>
@@
 <attribute name="VALUE" x="34.036" y="28.2321" size="1.27" layer="27" rot="R90"/>
 </element>
-<element name="R19" library="rcl" package="R0805" value="1M" x="37.465" y="29.21" smashed="yes" rot="R270">
+<element name="R19" library="rcl" package="R0805" value="220k" x="37.465" y="29.21" smashed="yes" rot="R270">
 <attribute name="ELECROW" value="C17514" x="37.465" y="29.21" size="1.778" layer="27" rot="R270" display="off"/>
 <attribute name="LCSC" value="C17514" x="37.465" y="29.21" size="1.778" layer="27" rot="R270" display="off"/>
@@
 </signal>
 </signals>
+<mfgpreviewcolors>
+<mfgpreviewcolor name="soldermaskcolor" color="0xC8008000"/>
+<mfgpreviewcolor name="silkscreencolor" color="0xFFFEFEFE"/>
+<mfgpreviewcolor name="backgroundcolor" color="0xFF282828"/>
+<mfgpreviewcolor name="coppercolor" color="0xFFFFBF00"/>
+<mfgpreviewcolor name="substratecolor" color="0xFF786E46"/>
+</mfgpreviewcolors>
 </board>
 </drawing>
