File: rpi3-shield/eagle/shield.sch (EAGLE design)
At the start: 8 parts, among them J1 RJ12STRAIGHT-I2C, J2 RJ12STRAIGHT-I2C, J3 RJ12STRAIGHT-I2C, J4 22-27-2061-06, J5 22-27-2061-06, J6 22-27-2061-06, J7 22-27-2061-06

Commit message: rpi3-shield: v1.0.0 submitted for production
Parts:
- added LED1: red, led:LEDSML0805
- added R1: 1k, rcl:R-EU_R0805
- added R2, R3: 10k, rcl:R-EU_R0805
Connections:
- new net IO13: LED1.A, PCB1.GPIO13
- new net IO17: J5-4.S, PCB1.GPIO17
- new net IO18: J4-4.S, PCB1.GPIO18
- new net IO19: J7-2.S, PCB1.GPIO19
- new net IO22: J5-2.S, PCB1.GPIO22
- new net IO27: J5-3.S, PCB1.GPIO27
- new net IO5: J7-4.S, PCB1.GPIO5
- new net IO6: J7-3.S, PCB1.GPIO6
- new net N$2: LED1.C, R1.1
- net +3V3: now also J1.1, J2.1, J3.1, J4-1.S, J5-1.S, J6-1.S, J7-1.S
- net +5V: now also J1.5, J2.5, J3.5, J4-5.S, J5-5.S, J6-5.S, J7-5.S, R2.1, R3.1
- net GND: now also J1.4, J1.6, J2.4, J2.6, J3.4, J3.6, J4-6.S, J5-6.S, J6-6.S, J7-6.S, R1.2
- net MISO0: now also J6-3.S
- net MOSI0: now also J6-4.S
- net RX: now also J4-3.S
- net SCL1: now also J1.2, J2.2, J3.2, R3.2
- net SCLK0: now also J6-2.S
- net SDA1: now also J1.3, J2.3, J3.3, R2.2
- net TX: now also J4-2.S
Other:
- moved on the sheet: J1, J2, J3, J4-1, J4-2, J4-3, J4-4, J4-5, J4-6, J5-1, J5-2, J5-3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
