File: counter-i2c/eagle/counter.sch (EAGLE design)
At the start: 76 parts, among them IC1 MCP1703DB, IC2 4067D, IC3 74HC154DW, J1 RJ12RIGHTANGLE-I2C, X2 8MHz, X4 MINI-USB

Commit message: master: fix parameter for logging interval
Connections:
- net A5: now also IC3A.G2
- net GND: no longer IC3A.G2
Other:
- moved on the sheet: IC3P
Changed lines of the file:
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@@
 <?xml version="1.0" encoding="utf-8"?>
 <!DOCTYPE eagle SYSTEM "eagle.dtd">
-<eagle version="9.0.0">
+<eagle version="9.1.0">
 <drawing>
 <settings>
@@
 <instance part="IC3" gate="A" x="91.44" y="208.28"/>
 <instance part="IC2" gate="P" x="337.82" y="195.58"/>
-<instance part="IC3" gate="P" x="68.58" y="195.58"/>
-<instance part="P+9" gate="G$1" x="68.58" y="203.2"/>
-<instance part="GND20" gate="1" x="68.58" y="182.88"/>
+<instance part="IC3" gate="P" x="53.34" y="193.04"/>
+<instance part="P+9" gate="G$1" x="53.34" y="200.66"/>
+<instance part="GND20" gate="1" x="53.34" y="180.34"/>
 <instance part="GND25" gate="1" x="337.82" y="185.42"/>
 <instance part="P+21" gate="G$1" x="337.82" y="203.2"/>
-<instance part="GND12" gate="1" x="78.74" y="180.34"/>
+<instance part="GND12" gate="1" x="73.66" y="180.34"/>
 <instance part="O3" gate="G$1" x="157.48" y="266.7" rot="R270"/>
 <instance part="RK5" gate="G$1" x="170.18" y="261.62" rot="R180"/>
@@
 <pinref part="IC3" gate="P" pin="GND"/>
 <pinref part="GND20" gate="1" pin="GND"/>
-<wire x1="68.58" y1="185.42" x2="68.58" y2="187.96" width="0.1524" layer="91"/>
+<wire x1="53.34" y1="182.88" x2="53.34" y2="185.42" width="0.1524" layer="91"/>
 </segment>
 <segment>
@@
 <segment>
 <pinref part="IC3" gate="A" pin="G1"/>
-<pinref part="IC3" gate="A" pin="G2"/>
-<wire x1="78.74" y1="190.5" x2="78.74" y2="187.96" width="0.1524" layer="91"/>
 <pinref part="GND12" gate="1" pin="GND"/>
-<wire x1="78.74" y1="182.88" x2="78.74" y2="187.96" width="0.1524" layer="91"/>
-<junction x="78.74" y="187.96"/>
+<wire x1="78.74" y1="190.5" x2="73.66" y2="190.5" width="0.1524" layer="91"/>
+<wire x1="73.66" y1="190.5" x2="73.66" y2="182.88" width="0.1524" layer="91"/>
 </segment>
 <segment>
@@
 <wire x1="469.9" y1="175.26" x2="485.14" y2="175.26" width="0.1524" layer="91"/>
 <label x="480.06" y="175.26" size="1.778" layer="95"/>
+</segment>
+<segment>
+<pinref part="IC3" gate="A" pin="G2"/>
+<wire x1="78.74" y1="187.96" x2="76.2" y2="187.96" width="0.1524" layer="91"/>
+<label x="76.2" y="187.96" size="1.778" layer="95"/>
 </segment>
 </net>
@@
 </sheet>
 </sheets>
+<errors>
+</errors>
 </schematic>
 </drawing>
