File: master/eagle/beemos-master.brd (EAGLE design)
At the start: 99.1 x 73.7 mm, 61 parts, among them CON1 BATTERY, CON2 JACK_DC_BARREL, CON3 SPI, IC1 32U4, IC2 MCP73831T, IC3 MCP1703CB, IC4 DMP1045U, J1 RJ12STRAIGHT-I2C, J2 RJ12STRAIGHT-I2C, J3 RJ12STRAIGHT-I2C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

Commit message: master: working on version 1.1 of PCB
Parts:
- added C12, C13: 10u, rcl:C0805K
- added C14: 100nF, rcl:C0805K
- added IC5: MCP1703-50, linear:SOT23
- moved U$1 77.5 mm to (74.2, 18.0)
- moved CON2 27.9 mm to (-0.64, 50.2)
- moved D3 23.6 mm to (44.5, 47.0), turned to 270 degrees
- moved R15 22.5 mm to (22.2, 38.1)
- moved R18 22.2 mm to (64.1, 52.7), turned to 180 degrees
- moved R19 19.8 mm to (64.1, 50.2), turned to 0 degrees
- moved R17 19.1 mm to (58.4, 48.9), turned to 0 degrees
- moved IC4 17.9 mm to (40.0, 47.0), turned to 90 degrees
- moved C11 17.9 mm to (64.1, 47.6), turned to 0 degrees
- moved C5 16.6 mm to (29.8, 48.9)
- moved D2 16.2 mm to (22.2, 41.3)
- moved R3 15.4 mm to (29.8, 40.0)
- moved IC2 15.4 mm to (29.8, 44.5)
- moved IC3 15.3 mm to (45.1, 36.2)
- moved CON3 15.1 mm to (65.4, 21.0), turned to 180 degrees
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Connections:
- new net N$12: C12.1, CON2.P$1, IC5.3
- net 3.3V: now also J1.+12V, J2.+12V, J3.+12V, J4.+12V, R1.2, R6.2
- net D12: now also JP1.1
- net GND: now also C12.2, C13.2, C14.2, IC5.1
- net N$3: now also C13.1, C14.1, IC5.2; no longer CON2.P$1
- net VBAT1: no longer JP1.2, X6.8
- net VDD: now also JP1.2, X6.8; no longer R1.2, R6.2
Routing:
- net VBAT1: track 151.4 -> 10.4 mm, vias 3 -> 0
- net VDD: track 136.6 -> 3.74 mm
- net 3.3V: track 180.5 -> 48.0 mm, vias 4 -> 0
- net GND: track 196.5 -> 81.5 mm, vias 24 -> 26
- net ISP+5V: track 115.0 -> 0.00 mm, vias 6 -> 0
- net SCL: track 140.9 -> 59.8 mm, vias 3 -> 0
- net VUSB: track 99.9 -> 20.9 mm
- net D6: track 74.6 -> 0.00 mm, vias 2 -> 0
- net SDA: track 132.2 -> 65.3 mm, vias 4 -> 0
- net D9: track 64.9 -> 0.00 mm, vias 2 -> 0
- net A0: track 54.6 -> 0.00 mm, vias 1 -> 0
- net D5: track 54.4 -> 0.00 mm, vias 1 -> 0
- net TX: track 52.6 -> 0.00 mm, vias 1 -> 0
- net A1: track 50.4 -> 0.00 mm, vias 1 -> 0
- net D10: track 76.9 -> 29.0 mm, vias 4 -> 1
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- added copper zone on layer 1, net VDD
Other:
- outline, holes or cut-outs redrawn
- board text added: "BeeMoS I2C master v1.1"
- board text added: "VDD"
- board text removed: "BeeMoS I2C master v1.0"
- board text removed: "VBAT1"

Commit message: master: pcb version 1.1
Parts:
- D1, D2, D4: value Schottky|| -> Schottky
- moved U$1 33.6 mm to (79.5, 51.2), turned to 90 degrees
- moved R1 4.96 mm to (94.0, 59.1), turned to 270 degrees
- moved R6 4.96 mm to (97.2, 59.1), turned to 270 degrees
- moved C6 1.80 mm to (43.8, 40.6)
- moved C7 1.80 mm to (43.8, 43.2)
- moved C8 1.80 mm to (43.8, 33.7)
- moved IC3 1.80 mm to (43.8, 37.5)
- moved C10 1.80 mm to (50.8, 38.7)
- moved C3 1.80 mm to (50.8, 34.9)
- moved D3 1.27 mm to (44.5, 48.3)
- moved IC4 1.27 mm to (40.0, 48.3)
Routing:
- net 3.3V: track 48.0 -> 215.9 mm, vias 0 -> 8
- net VDD: track 3.74 -> 93.2 mm, vias 0 -> 2
- net ISP+5V: track 0.00 -> 70.0 mm, vias 0 -> 2
- net D12: track 0.00 -> 69.0 mm, vias 0 -> 2
- net D6: track 0.00 -> 64.3 mm, vias 0 -> 2
- net VUSB: track 20.9 -> 80.7 mm
- net VBAT1: track 10.4 -> 67.9 mm
- net TX: track 0.00 -> 52.1 mm
- net RX: track 0.00 -> 45.0 mm
- net SCL: track 59.8 -> 103.6 mm, vias 0 -> 2
- net A3: track 0.00 -> 36.8 mm, vias 0 -> 1
- net A2: track 0.00 -> 36.2 mm, vias 0 -> 1
- net A1: track 0.00 -> 35.4 mm, vias 0 -> 1
- net A0: track 0.00 -> 34.9 mm, vias 0 -> 1
- net D5: track 0.00 -> 33.2 mm, vias 0 -> 1
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Other:
- board text added: "D12"
- board text added: "D6"
- board text added: "RX"
- board text added: "TX"
