File: master/eagle/beemos-master.sch (EAGLE design)
At the start: 61 parts, among them CON1 BATTERY, CON2 JACK_DC_BARREL, CON3 SPI, IC1 32U4, IC2 MCP73831T, IC3 MCP1703CB, IC4 DMP1045U, J1 RJ12STRAIGHT-I2C, J2 RJ12STRAIGHT-I2C, J3 RJ12STRAIGHT-I2C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

Commit message: master: working on version 1.1 of PCB
Parts:
- added C12, C13: 10u, rcl:C-EUC0805K
- added C14: 100nF, rcl:C-EUC0805K
- added IC5: MCP1703-50, linear:MCP1703CB
Connections:
- new net N$12: C12.1, CON2.V+, IC5.VI
- net 3.3V: now also J1.1, J2.1, J3.1, J4.1, R1.2, R6.2
- net D12: now also JP1.1
- net GND: now also C12.2, C13.2, C14.2, IC5.GND
- net N$3: now also C13.1, C14.1, IC5.VO; no longer CON2.V+
- net VBAT1: no longer JP1.2, X6-8.S
- net VDD: now also JP1.2, X6-8.S; no longer R1.2, R6.2
Other:
- note added: "5.0V LDO"
- note removed: "Over voltage protection * Consumption ? * Check resistance"
- moved on the sheet: D4

Commit message: master: pcb version 1.1
Parts:
- D1, D2, D4: value Schottky|| -> Schottky
Changed lines of the file:
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@@
 </part>
 <part name="SUPPLY3" library="supply1" library_urn="urn:adsk.eagle:library:371" deviceset="VDD" device=""/>
-<part name="P+1" library="supply1" library_urn="urn:adsk.eagle:library:371" deviceset="VCC" device=""/>
 <part name="IC4" library="dp_devices" deviceset="TRANSISTOR_FET_TSM2301CX" device="" value="DMP1045U">
 <attribute name="LCSC" value="C96613"/>
@@
 <part name="SUPPLY4" library="supply1" library_urn="urn:adsk.eagle:library:371" deviceset="VDD" device=""/>
 <part name="U$2" library="MyPOW" deviceset="VUSB" device=""/>
-<part name="D1" library="diode" library_urn="urn:adsk.eagle:library:210" deviceset="MBR0520LT" device="" package3d_urn="urn:adsk.eagle:package:43420/1" value="Schottky||">
+<part name="D1" library="diode" library_urn="urn:adsk.eagle:library:210" deviceset="MBR0520LT" device="" package3d_urn="urn:adsk.eagle:package:43420/1" value="Schottky">
 <attribute name="LCSC" value="C82544"/>
 <attribute name="MPN" value="621-1N5819HW-F"/>
 </part>
-<part name="D2" library="diode" library_urn="urn:adsk.eagle:library:210" deviceset="MBR0520LT" device="" package3d_urn="urn:adsk.eagle:package:43420/1" value="Schottky||">
+<part name="D2" library="diode" library_urn="urn:adsk.eagle:library:210" deviceset="MBR0520LT" device="" package3d_urn="urn:adsk.eagle:package:43420/1" value="Schottky">
 <attribute name="LCSC" value="C82544"/>
 <attribute name="MPN" value="621-1N5819HW-F"/>
@@
 <part name="J4" library="lpatiny" deviceset="RJ12" device="STRAIGHT-I2C" value="RJ12STRAIGHT-I2C"/>
 <part name="CON2" library="lpatiny" deviceset="JACK_DC_BARREL" device=""/>
-<part name="D4" library="diode" library_urn="urn:adsk.eagle:library:210" deviceset="MBR0520LT" device="" package3d_urn="urn:adsk.eagle:package:43420/1" value="Schottky||">
+<part name="D4" library="diode" library_urn="urn:adsk.eagle:library:210" deviceset="MBR0520LT" device="" package3d_urn="urn:adsk.eagle:package:43420/1" value="Schottky">
 <attribute name="LCSC" value="C82544"/>
 <attribute name="MPN" value="621-1N5819HW-F"/>
@@
 </part>
 <part name="IC5" library="linear" library_urn="urn:adsk.eagle:library:262" deviceset="MCP1703" device="CB" package3d_urn="urn:adsk.eagle:package:16489/2" value="MCP1703-50"/>
+<part name="P+1" library="SparkFun" deviceset="3.3V" device=""/>
 </parts>
 <sheets>
@@
 </instance>
 <instance part="SUPPLY3" gate="G$1" x="-7.62" y="53.34"/>
-<instance part="P+1" gate="VCC" x="25.4" y="53.34"/>
 <instance part="IC4" gate="G$1" x="157.48" y="104.14" rot="MR270">
 <attribute name="MPN" x="157.48" y="104.14" size="1.778" layer="96" rot="MR270" display="off"/>
@@
 </instance>
 <instance part="IC5" gate="G$1" x="-45.72" y="106.68"/>
+<instance part="P+1" gate="G$1" x="25.4" y="50.8"/>
 </instances>
 <busses>
@@
 <junction x="25.4" y="45.72"/>
 <pinref part="C6" gate="G$1" pin="1"/>
-<pinref part="P+1" gate="VCC" pin="VCC"/>
 <wire x1="25.4" y1="45.72" x2="25.4" y2="50.8" width="0.1524" layer="91"/>
 <pinref part="C7" gate="G$1" pin="1"/>
@@
 <pinref part="IC3" gate="G$1" pin="VO"/>
 <wire x1="20.32" y1="45.72" x2="25.4" y2="45.72" width="0.1524" layer="91"/>
+<pinref part="P+1" gate="G$1" pin="3.3V"/>
 </segment>
 <segment>
@@
 <wire x1="-73.152" y1="106.68" x2="-63.5" y2="106.68" width="0.1524" layer="91"/>
 <junction x="-73.152" y="106.68"/>
-</segment>
-</net>
+<junction x="-63.5" y="106.68"/>
+</segment>
+</net>
