File: lcd-screen-i2c/eagle/lcd-screen.sch (EAGLE design)
At the start: 29 parts, among them CON1 SPI, IC1 MCP1703CB, J1 RJ12RIGHTANGLE-I2C, J2 RJ12RIGHTANGLE-I2C, J3 RJ12RIGHTANGLE-I2C, U1 ATMEGA328P_TQFP, X1 8MHz

Commit message: Change rotary encoder pinout to use interruptible pins on Atmega328p
Connections:
- net D3: now also U$1.GND; no longer U$1.INT
- net D4: now also U$1.INT; no longer U$1.B
- net GND: now also U$1.B; no longer U$1.GND
Changed lines of the file:
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@@
 </instance>
 <instance part="U$1" gate="G$1" x="30.48" y="27.94"/>
-<instance part="GND10" gate="1" x="22.86" y="17.78"/>
+<instance part="GND10" gate="1" x="17.78" y="25.4"/>
 <instance part="GND12" gate="1" x="48.26" y="33.02"/>
 <instance part="D1" gate="G$1" x="68.58" y="185.42">
@@
 </segment>
 <segment>
-<pinref part="U$1" gate="G$1" pin="GND"/>
-<pinref part="GND10" gate="1" pin="GND"/>
-</segment>
-<segment>
 <pinref part="U$1" gate="G$1" pin="CLSD"/>
 <pinref part="GND12" gate="1" pin="GND"/>
@@
 <pinref part="GND39" gate="1" pin="GND"/>
 <junction x="93.98" y="93.98"/>
+</segment>
+<segment>
+<pinref part="U$1" gate="G$1" pin="B"/>
+<pinref part="GND10" gate="1" pin="GND"/>
+<wire x1="22.86" y1="27.94" x2="17.78" y2="27.94" width="0.1524" layer="91"/>
 </segment>
 </net>
@@
 <pinref part="U$1" gate="G$1" pin="A"/>
 <wire x1="17.78" y1="35.56" x2="22.86" y2="35.56" width="0.1524" layer="91"/>
-<label x="20.32" y="35.56" size="1.778" layer="95" rot="R90"/>
+<label x="20.32" y="38.1" size="1.778" layer="95" rot="R180"/>
 </segment>
 </net>
@@
 </segment>
 <segment>
-<pinref part="U$1" gate="G$1" pin="INT"/>
-<wire x1="55.88" y1="20.32" x2="48.26" y2="20.32" width="0.1524" layer="91"/>
-<label x="50.8" y="17.78" size="1.778" layer="95"/>
+<pinref part="U$1" gate="G$1" pin="GND"/>
+<wire x1="22.86" y1="20.32" x2="17.78" y2="20.32" width="0.1524" layer="91"/>
+<label x="17.78" y="17.78" size="1.778" layer="95"/>
 </segment>
 </net>
@@
 </segment>
 <segment>
-<pinref part="U$1" gate="G$1" pin="B"/>
-<wire x1="22.86" y1="27.94" x2="17.78" y2="27.94" width="0.1524" layer="91"/>
-<label x="20.32" y="27.94" size="1.778" layer="95" rot="R90"/>
-</segment>
-</net>
+<pinref part="U$1" gate="G$1" pin="INT"/>
+<wire x1="48.26" y1="20.32" x2="53.34" y2="20.32" width="0.1524" layer="91"/>
+<label x="50.8" y="17.78" size="1.778" layer="95"/>
+</segment>
+</net>
